File: Proyecto/diseño Eagle/Sistema SCADA.sch (EAGLE design)
At the start: 31 parts, among them Q1 2N3565, Q2 2N3565, Q3 2N3565, Q4 2N3565, Q5 2N3565, X1 SMKDSP_1,5/2, X10 SMKDSP_1,5/2, X11 SMKDSP_1,5/6, X12 SMKDSP_1,5/2, X13 SMKDSP_1,5/2, X14 SMKDSP_1,5/2, X2 SMKDSP_1,5/3, X3 SMKDSP_1,5/4, X4 SMKDSP_1,5/4, X5 SMKDSP_1,5/4, X6 SMKDSP_1,5/4, X7 SMKDSP_1,5/3, X8 SMKDSP_1,5/2, X9 SMKDSP_1,5/2

Commit message: Major changes
Parts:
- removed Q1, Q2, Q3, Q4, Q5: 2N3565, transistor-npn:2N3565
- removed R1, R10, R11, R2, R3, R4, R5, R6, R7, R8, R9: (no value), resistor:R-EU_0207/10
- removed X10, X12, X13, X14, X8, X9: SMKDSP_1,5/2, con-phoenix-smkdsp:SMKDSP_1,5/2
- removed X4, X5, X6: SMKDSP_1,5/4, con-phoenix-smkdsp:SMKDSP_1,5/4
- removed X7: SMKDSP_1,5/3, con-phoenix-smkdsp:SMKDSP_1,5/3
- added K1, K2, K3, K4, K5, K6, K7, K8: 35701331, relay:35701331
Connections:
- removed net N$1: Q1.B, R1.2
- removed net N$10: Q4.B, R7.2
- removed net N$11: Q4.E, R8.1
- removed net N$12: Q4.C, X10-1.KL
- removed net N$13: PCB1.2, X12-1.KL
- removed net N$14: PCB1.5V, X11-2.KL, X13-2.KL, X2-3.KL, X3-4.KL, X4-4.KL, X5-4.KL, X6-4.KL, X7-3.KL
- removed net N$15: PCB1.11, X4-3.KL
- removed net N$16: X1-2.KL, X10-2.KL, X14-2.KL, X8-2.KL, X9-2.KL
- removed net N$17: PCB1.14(TX3), R3.1
- removed net N$18: PCB1.15(RX3), R5.1
- removed net N$19: PCB1.16(TX2), R7.1
- removed net N$2: Q1.E, R2.1
- removed net N$20: PCB1.13, X3-3.KL
- removed net N$21: PCB1.12, X3-2.KL
- removed net N$22: R9.1, X12-2.KL
- removed net N$23: PCB1.7, X6-3.KL
- removed net N$24: PCB1.0(RX), X11-4.KL
- removed net N$25: PCB1.10, X4-2.KL
- removed net N$26: PCB1.1(TX), X11-5.KL
- removed net N$27: PCB1.9, X5-3.KL
- removed net N$28: PCB1.8, X5-2.KL
- removed net N$29: Q5.B, R10.2
- removed net N$3: Q1.C, X1-1.KL
- removed net N$30: PCB1.6, X6-2.KL
- removed net N$31: PCB1.5, X2-2.KL
- removed net N$32: PCB1.4, X7-2.KL
- removed net N$33: PCB1.3, R1.1
- removed net N$35: Q5.E, R11.1
- removed net N$36: Q5.C, X14-1.KL
- removed net N$37: PCB1.17(RX2), R10.1
- removed net N$39: PCB1.GND, R11.2, R2.2, R4.2, R6.2, R8.2, R9.2, X11-3.KL, X13-1.KL, X2-1.KL, X3-1.KL, X4-1.KL, X5-1.KL, X6-1.KL, X7-1.KL
- removed net N$4: Q2.B, R3.2
- removed net N$5: Q2.E, R4.1
- removed net N$6: Q2.C, X8-1.KL
- removed net N$7: Q3.B, R5.2
- removed net N$8: Q3.E, R6.1
- removed net N$9: Q3.C, X9-1.KL
Other:
- moved on the sheet: X1-1, X1-2, X11-1, X11-2, X11-3, X11-4, X11-5, X11-6, X2-1, X2-2, X2-3, X3-1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
